File: el_wirecontroller.brd (EAGLE design)
At the start: 100 x 80 mm, 13 parts, among them U1 Tiny45-20-SMT

Commit message: add transistor
Parts:
- added Q1: (no value), adafruit:SOT23
- added R4: 2M, SparkFun-Passives:0402-RES
- moved C2 8.71 mm to (14.6, 11.7), turned to 180 degrees
- moved C1 1.46 mm to (26.4, 9.25), turned to 180 degrees
Connections:
- new net N$14: Q1.3, R4.2
- new net N$3: Q1.1, U$1.P13
- net GND: now also Q1.2; no longer U$1.P13
- net VDD: now also R4.1
Routing:
- net N$3: track 0.00 -> 3.67 mm
- net N$7: track 11.6 -> 14.9 mm
- net N$14: track 0.00 -> 2.55 mm
- net VDD: track 51.1 -> 53.2 mm
- net GND: track 19.9 -> 19.2 mm
- net N$6: track 7.27 -> 7.30 mm, vias 1 -> 0
Changed lines of the file:
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@@
 <element name="U$1" library="blake_custom" package="QFN-16" value="HV861" x="19.14" y="16.36"/>
 <element name="R1" library="SparkFun-Passives" package="0402-RES" value="2M" x="15.25" y="15.7" rot="R180"/>
-<element name="C1" library="SparkFun-Passives" package="0402-CAP" value="3.3n" x="25.15" y="10" rot="R270"/>
+<element name="C1" library="SparkFun-Passives" package="0402-CAP" value="3.3n" x="26.4" y="9.25" rot="R180"/>
 <element name="D1" library="adafruit" package="DO-1N4148" value="1N4148" x="26" y="6.85"/>
 <element name="R2" library="SparkFun-Passives" package="0402-RES" value="825k" x="15.3" y="14.3" rot="R180"/>
-<element name="C2" library="SparkFun-Passives" package="0402-CAP" value="0.1u" x="14.9" y="20.4"/>
+<element name="C2" library="SparkFun-Passives" package="0402-CAP" value="0.1u" x="14.6" y="11.7" rot="R180"/>
 <element name="R3" library="SparkFun-Passives" package="0402-RES" value="3.3M" x="18.5" y="18.55" rot="R180"/>
 <element name="C3" library="SparkFun-Passives" package="0402-CAP" value="2.2u" x="14.9" y="18.55" rot="R180"/>
@@
 <element name="JP3" library="SparkFun-Connectors" package="1X02" value="M02PTH" x="29.6" y="17.35" rot="R90"/>
 <element name="JP4" library="pinhead" package="2X03" value="" x="7.8" y="16.4" rot="R90"/>
+<element name="Q1" library="adafruit" package="SOT23" value="" x="20.9" y="20.5" rot="R90"/>
+<element name="R4" library="SparkFun-Passives" package="0402-RES" value="2M" x="16.6" y="20.5"/>
 </elements>
 <signals>
@@
 <wire x1="6.6" y1="20.4" x2="11.2" y2="20.4" width="0.3048" layer="1"/>
 <contactref element="JP1" pad="2"/>
-<wire x1="11.2" y1="20.4" x2="14.25" y2="20.4" width="0.3048" layer="1"/>
 <wire x1="11.2" y1="12.8" x2="11.2" y2="15" width="0.3048" layer="1"/>
 <wire x1="19.44" y1="14.61" x2="19.01" y2="14.61" width="0.3048" layer="1"/>
@@
 <wire x1="11.2" y1="15" x2="14.6" y2="15" width="0.3048" layer="1"/>
 <contactref element="JP4" pad="2"/>
-<wire x1="15.3" y1="5.245" x2="15.3" y2="12.8" width="0.3048" layer="1"/>
+<wire x1="15.3" y1="5.245" x2="15.3" y2="11.7" width="0.3048" layer="1"/>
+<wire x1="15.3" y1="11.7" x2="15.3" y2="12.8" width="0.3048" layer="1"/>
 <wire x1="12.7472" y1="5.245" x2="15.3" y2="5.245" width="0.3048" layer="1"/>
 <wire x1="4.9" y1="20.4" x2="4.9" y2="15.49" width="0.3048" layer="1"/>
 <wire x1="4.9" y1="15.49" x2="6.53" y2="13.86" width="0.3048" layer="1"/>
-<wire x1="6.66" y1="23.35" x2="6.66" y2="20.46" width="0.3048" layer="1"/>
 <wire x1="6.66" y1="20.46" x2="6.6" y2="20.4" width="0.3048" layer="1"/>
 <wire x1="11.2" y1="15" x2="11.2" y2="20.4" width="0.3048" layer="1"/>
 <wire x1="6.6" y1="20.4" x2="4.9" y2="20.4" width="0.3048" layer="1"/>
+<contactref element="R4" pad="1"/>
+<wire x1="6.66" y1="23.35" x2="6.66" y2="20.46" width="0.3048" layer="1"/>
+<wire x1="15.25" y1="11.7" x2="15.3" y2="11.7" width="0.3048" layer="1"/>
+<wire x1="11.2" y1="20.4" x2="16.1" y2="20.4" width="0.3048" layer="1"/>
+<wire x1="16.1" y1="20.4" x2="15.95" y2="20.5" width="0.3048" layer="1"/>
 </signal>
 <signal name="N$6">
@@
 <contactref element="D1" pad="A"/>
 <wire x1="20.94" y1="13.61" x2="20.95" y2="13.61" width="0.3048" layer="1"/>
-<via x="21.75" y="11.4" extent="1-16" drill="0.6" shape="square"/>
-<wire x1="21.75" y1="11.4" x2="21.7" y2="11.4" width="0.3048" layer="16"/>
-<wire x1="22.19" y1="6.85" x2="21.75" y2="8.55" width="0.4064" layer="16"/>
-<wire x1="21.75" y1="8.55" x2="21.75" y2="11.4" width="0.4064" layer="16"/>
-<wire x1="21.75" y1="11.4" x2="21.65" y2="11.4" width="0.3048" layer="1"/>
-<wire x1="21.65" y1="11.4" x2="20.95" y2="12.1" width="0.3048" layer="1"/>
-<wire x1="20.95" y1="12.1" x2="20.95" y2="13.6" width="0.3048" layer="1"/>
-<wire x1="20.95" y1="13.6" x2="20.94" y2="13.61" width="0.3048" layer="1"/>
+<wire x1="20.94" y1="13.61" x2="20.94" y2="10.66" width="0.3048" layer="1"/>
+<wire x1="20.94" y1="10.66" x2="22.2" y2="9.4" width="0.3048" layer="1"/>
+<wire x1="22.2" y1="9.4" x2="22.2" y2="6.86" width="0.3048" layer="1"/>
+<wire x1="22.2" y1="6.86" x2="22.19" y2="6.85" width="0.3048" layer="1"/>
 </signal>
 <signal name="N$7">
@@
 <wire x1="29.81" y1="6.85" x2="29.45" y2="6.85" width="0.3048" layer="1"/>
 <wire x1="21.44" y1="13.61" x2="21.44" y2="13.56" width="0.3048" layer="1"/>
-<wire x1="21.44" y1="13.56" x2="24.3" y2="10.7" width="0.3048" layer="1"/>
-<wire x1="24.3" y1="10.7" x2="25.2" y2="10.7" width="0.3048" layer="1"/>
-<wire x1="25.2" y1="10.7" x2="25.96" y2="10.7" width="0.3048" layer="1"/>
-<wire x1="25.96" y1="10.7" x2="29.81" y2="6.85" width="0.3048" layer="1"/>
-<wire x1="25.15" y1="10.65" x2="25.2" y2="10.7" width="0.3048" layer="1"/>
+<wire x1="21.44" y1="13.56" x2="21.5" y2="13.56" width="0.3048" layer="1"/>
+<wire x1="21.5" y1="13.56" x2="21.5" y2="10.9" width="0.3048" layer="1"/>
+<wire x1="21.5" y1="10.9" x2="24.7" y2="8.2" width="0.3048" layer="1"/>
+<wire x1="29.45" y1="6.85" x2="29.45" y2="6.95" width="0.3048" layer="1"/>
+<wire x1="29.45" y1="6.95" x2="28.1" y2="8.2" width="0.3048" layer="1"/>
+<wire x1="28.1" y1="8.2" x2="24.7" y2="8.2" width="0.3048" layer="1"/>
+<wire x1="28.1" y1="8.2" x2="27.2" y2="9.1" width="0.3048" layer="1"/>
+<wire x1="27.05" y1="9.25" x2="27.2" y2="9.1" width="0.3048" layer="1"/>
+<wire x1="27.2" y1="9.1" x2="27.2" y2="9.2" width="0.3048" layer="1"/>
+<wire x1="27.2" y1="9.2" x2="27" y2="9.4" width="0.3048" layer="1"/>
+<wire x1="27" y1="9.4" x2="27.1" y2="9.4" width="0.3048" layer="1"/>
+<wire x1="27.1" y1="9.4" x2="27.1" y2="9.1" width="0.3048" layer="1"/>
 </signal>
 <signal name="GND">
 <contactref element="C1" pad="2"/>
-<contactref element="U$1" pad="P13"/>
 <contactref element="C2" pad="2"/>
 <contactref element="U$1" pad="P6"/>
@@
 <wire x1="20.45" y1="14.15" x2="20.49" y2="14.85" width="0.3048" layer="1"/>
 <wire x1="20.49" y1="14.85" x2="20.69" y2="14.86" width="0.3048" layer="1"/>
-<wire x1="21.45" y1="16.11" x2="21.3" y2="15.07" width="0.3048" layer="1"/>
-<wire x1="21.3" y1="15.07" x2="20.69" y2="14.86" width="0.3048" layer="1"/>
 <contactref element="U1" pad="4"/>
 <polygon width="0.3048" layer="16">
@@
 <wire x1="20.45" y1="13.61" x2="20.45" y2="10.65" width="0.3048" layer="1"/>
 <wire x1="20.45" y1="10.65" x2="19.8" y2="10.2" width="0.3048" layer="1"/>
-<via x="21.45" y="18.7" extent="1-16" drill="0.6" shape="square"/>
-<wire x1="21.45" y1="18.7" x2="21.35" y2="18.6" width="0.3048" layer="16"/>
-<wire x1="21.45" y1="18.7" x2="21.35" y2="18.7" width="0.3048" layer="1"/>
-<wire x1="21.45" y1="18.7" x2="21.45" y2="16.11" width="0.3048" layer="1"/>
-<wire x1="21.45" y1="16.05" x2="21.45" y2="16.11" width="0.3048" layer="1"/>
-<wire x1="21.44" y1="16.11" x2="21.45" y2="16.11" width="0.3048" layer="1"/>
 <contactref element="JP1" pad="1"/>
 <wire x1="14.25" y1="18.55" x2="14.2" y2="18.55" width="0.3048" layer="1"/>
 <via x="12.4" y="18.6" extent="1-16" drill="0.6" shape="square"/>
 <wire x1="12.4" y1="18.6" x2="14.3" y2="17.3" width="0.3048" layer="16"/>
-<wire x1="25.15" y1="9.35" x2="25.15" y2="7.65" width="0.3048" layer="1"/>
-<wire x1="25.15" y1="7.65" x2="25.2" y2="7.6" width="0.3048" layer="1"/>
-<wire x1="25.2" y1="7.6" x2="25.1" y2="7.6" width="0.3048" layer="1"/>
-<via x="25.1" y="7.6" extent="1-16" drill="0.6" shape="square"/>
-<wire x1="25.1" y1="7.6" x2="25.2" y2="7.6" width="0.3048" layer="16"/>
 <contactref element="JP4" pad="6"/>
 <wire x1="12.4" y1="18.6" x2="14.2" y2="18.6" width="0.3048" layer="1"/>
 <wire x1="14.2" y1="18.6" x2="14.25" y2="18.55" width="0.3048" layer="1"/>
-<wire x1="15.55" y1="20.4" x2="17.6" y2="20.4" width="0.3048" layer="1"/>
-<via x="17.6" y="20.4" extent="1-16" drill="0.6" shape="square"/>
-<wire x1="17.6" y1="20.4" x2="17.7" y2="20.4" width="0.3048" layer="16"/>
+<contactref element="Q1" pad="2"/>
+<wire x1="22" y1="21.45" x2="22" y2="23.1" width="0.3048" layer="1"/>
+<wire x1="22" y1="23.15" x2="22" y2="23.1" width="0.3048" layer="1"/>
+<via x="22" y="23.1" extent="1-16" drill="0.6" shape="square"/>
+<wire x1="22" y1="23.1" x2="23.3" y2="23.1" width="0.3048" layer="16"/>
+<wire x1="13.95" y1="11.7" x2="12" y2="11.7" width="0.3048" layer="1"/>
+<via x="12" y="11.7" extent="1-16" drill="0.6" shape="square"/>
+<wire x1="12" y1="11.7" x2="12.8" y2="10.4" width="0.3048" layer="16"/>
+<wire x1="25.75" y1="9.25" x2="25.7" y2="9.25" width="0.3048" layer="1"/>
+<wire x1="25.7" y1="9.25" x2="25.7" y2="10.5" width="0.3048" layer="1"/>
+<via x="25.7" y="10.5" extent="1-16" drill="0.6" shape="square"/>
+<wire x1="25.7" y1="10.5" x2="25.6" y2="10.5" width="0.3048" layer="16"/>
+<wire x1="25.6" y1="10.5" x2="25.6" y2="10.6" width="0.3048" layer="16"/>
 </signal>
 <signal name="N$9">
@@
 <wire x1="7.63" y1="17.5" x2="6.53" y2="16.4" width="0.3048" layer="1"/>
 </signal>
+<signal name="N$3">
+<contactref element="U$1" pad="P13"/>
+<contactref element="Q1" pad="1"/>
+<wire x1="21.44" y1="16.11" x2="21.44" y2="16.74" width="0.3048" layer="1"/>
+<wire x1="21.44" y1="16.74" x2="22" y2="17.3" width="0.3048" layer="1"/>
+<wire x1="22" y1="17.3" x2="22" y2="19.55" width="0.3048" layer="1"/>
+</signal>
+<signal name="N$14">
+<contactref element="Q1" pad="3"/>
+<contactref element="R4" pad="2"/>
+<wire x1="19.8" y1="20.5" x2="17.25" y2="20.5" width="0.3048" layer="1"/>
+</signal>
 </signals>
