File: el_wirecontroller.sch (EAGLE design)
At the start: 13 parts, among them U1 Tiny45-20-SMT

Commit message: add transistor
Parts:
- added Q1: (no value), adafruit:MOSFET-NREFLOW
- added R4: 2M, SparkFun-Passives:RESISTOR0402-RES
Connections:
- new net N$14: Q1.D, R4.2
- new net N$3: Q1.G, U$1.PWM
- net GND: now also Q1.S; no longer U$1.PWM
- net VDD: now also R4.1
Changed lines of the file:
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@@
 <part name="GND6" library="SparkFun-Aesthetics" deviceset="GND" device=""/>
 <part name="JP4" library="pinhead" deviceset="PINHD-2X3" device=""/>
+<part name="Q1" library="adafruit" deviceset="MOSFET-N" device="REFLOW"/>
+<part name="R4" library="SparkFun-Passives" deviceset="RESISTOR" device="0402-RES" value="2M"/>
 </parts>
 <sheets>
@@
 <instance part="GND6" gate="1" x="5.08" y="78.74"/>
 <instance part="JP4" gate="A" x="124.46" y="86.36"/>
+<instance part="Q1" gate="G$1" x="106.68" y="48.26"/>
+<instance part="R4" gate="G$1" x="109.22" y="60.96" rot="R270"/>
 </instances>
 <busses>
@@
 <label x="137.16" y="88.9" size="1.778" layer="95"/>
 </segment>
+<segment>
+<pinref part="R4" gate="G$1" pin="1"/>
+<wire x1="109.22" y1="66.04" x2="109.22" y2="71.12" width="0.1524" layer="91"/>
+<label x="109.22" y="71.12" size="1.778" layer="95"/>
+</segment>
 </net>
 <net name="GND" class="0">
@@
 <segment>
 <pinref part="GND4" gate="1" pin="GND"/>
-<pinref part="U$1" gate="G$1" pin="PWM"/>
-<wire x1="53.34" y1="45.72" x2="86.36" y2="45.72" width="0.1524" layer="91"/>
-<wire x1="86.36" y1="45.72" x2="86.36" y2="30.48" width="0.1524" layer="91"/>
+<wire x1="86.36" y1="30.48" x2="86.36" y2="25.4" width="0.1524" layer="91"/>
 <pinref part="C3" gate="G$1" pin="2"/>
-<wire x1="86.36" y1="30.48" x2="86.36" y2="25.4" width="0.1524" layer="91"/>
 <wire x1="73.66" y1="30.48" x2="86.36" y2="30.48" width="0.1524" layer="91"/>
+<pinref part="Q1" gate="G$1" pin="S"/>
+<wire x1="109.22" y1="43.18" x2="109.22" y2="30.48" width="0.1524" layer="91"/>
+<wire x1="109.22" y1="30.48" x2="86.36" y2="30.48" width="0.1524" layer="91"/>
 </segment>
 <segment>
@@
 </segment>
 </net>
+<net name="N$3" class="0">
+<segment>
+<pinref part="U$1" gate="G$1" pin="PWM"/>
+<wire x1="53.34" y1="45.72" x2="104.14" y2="45.72" width="0.1524" layer="91"/>
+<pinref part="Q1" gate="G$1" pin="G"/>
+</segment>
+</net>
+<net name="N$14" class="0">
+<segment>
+<pinref part="Q1" gate="G$1" pin="D"/>
+<pinref part="R4" gate="G$1" pin="2"/>
+<wire x1="109.22" y1="53.34" x2="109.22" y2="55.88" width="0.1524" layer="91"/>
+</segment>
+</net>
